Commit message: added laser

File: my_robot_description/urdf/camera.xacro (robot description, xacro)
@@ -24,5 +24,5 @@
         <sensor name="camera_sensor" type="camera">
             <pose>0 0 0 0 0 0</pose>
-            <visualize>true</visualize>
+            <visualize>false</visualize>
             <update_rate>10.0</update_rate>
             <plugin name="Camera_name" filename="libgazebo_ros_camera.so">

File: my_robot_description/urdf/common_properties.xacro (robot description, xacro)
@@ -6,4 +6,7 @@
   <material name="grey">
     <color rgba="0.5 0.5 0.5 1"/>
+  </material>
+  <material name="red">
+    <color rgba="1.0 0 0 1.0"/>
   </material>
   <xacro:macro name="box_inertia" params="m l w h xyz rpy">

File: my_robot_description/urdf/my_robot.urdf.xacro (robot description, xacro)
@@ -5,3 +5,4 @@
   <xacro:include filename="mobile_base_gazebo.xacro" />
   <xacro:include filename="camera.xacro" />
+  <xacro:include filename="lidar.xacro" />
 </robot>

Commit message: made changes to camera and fixed rotation issues

File: my_robot_description/urdf/camera.xacro (robot description, xacro)
@@ -20,12 +20,31 @@
         <origin xyz="0.305 0 0.1" rpy="0 0 0"/>
     </joint>
+    <joint name="camera_optical_joint" type="fixed">
+        <parent link="camera_link"/>
+        <child link="camera_link_optical"/>
+        <origin xyz="0 0 0" rpy="${-pi/2} 0 ${-pi/2}"/>
+    </joint>
+    <link name="camera_link_optical">
+    </link>
     <gazebo reference="camera_link">
         <material>Gazebo/Red</material>
-        <sensor name="camera_sensor" type="camera">
-            <pose>0 0 0 0 0 0</pose>
-            <visualize>false</visualize>
-            <update_rate>10.0</update_rate>
-            <plugin name="Camera_name" filename="libgazebo_ros_camera.so">
-                <frame_name>camera_link</frame_name>
+        <sensor name="camera" type="camera">
+            <pose> 0 0 0 0 0 0 </pose>
+            <visualize>true</visualize>
+            <update_rate>10</update_rate>
+            <camera>
+                <horizontal_fov>1.089</horizontal_fov>
+                <image>
+                    <format>R8G8B8</format>
+                    <width>640</width>
+                    <height>480</height>
+                </image>
+                <clip>
+                    <near>0.05</near>
+                    <far>8.0</far>
+                </clip>
+            </camera>
+            <plugin name="camera_controller" filename="libgazebo_ros_camera.so">
+                <frame_name>camera_link_optical</frame_name>
             </plugin>
         </sensor>
